File: rpiz_pi_platter/rpiz_pi_platter.kicad_pcb (KiCad board)
At the start: 2 copper layers, 65 x 30 mm, 7 parts, among them J1 GPIO_CONNECTOR, J2 BME680_CONNECTOR, J3 RFM95W_CONNECTOR

Commit message: modification of ground plane
Routing:
- net +5V: track 4.65 -> 2.60 mm
- net GND: track 79.1 -> 80.6 mm
Changed lines of the file:
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@@
   )
   (layers
-    (0 F.Cu signal hide)
+    (0 F.Cu signal)
     (31 B.Cu signal)
     (32 B.Adhes user)
@@
   (segment (start 146.222 95.838) (end 144.952 94.568) (width 0.25) (layer B.Cu) (net 1))
   (segment (start 125.902 93.298) (end 128.442 93.298) (width 0.25) (layer B.Cu) (net 2))
-  (segment (start 125.902 93.298) (end 123.846758 93.298) (width 0.25) (layer B.Cu) (net 2))
   (segment (start 123.846758 93.298) (end 123.833769 93.356311) (width 0.25) (layer B.Cu) (net 2))
   (segment (start 128.442 105.788) (end 128.652 105.998) (width 0.25) (layer B.Cu) (net 3))
@@
   (segment (start 171.832 108.538) (end 171.832 105.998) (width 0.25) (layer B.Cu) (net 5))
   (segment (start 136.272 105.998) (end 136.272 108.538) (width 0.25) (layer B.Cu) (net 5))
+  (segment (start 130.982 93.298) (end 129.922 92.238) (width 0.25) (layer B.Cu) (net 5))
   (segment (start 146.432 108.538) (end 143.682 105.788) (width 0.25) (layer B.Cu) (net 12))
   (segment (start 166.752 107.268) (end 165.482 108.538) (width 0.25) (layer B.Cu) (net 12))
