File: pi_platter_pcb/rpiz_pi_platter.kicad_pcb (KiCad board)
At the start: 2 copper layers, 65 x 30 mm, 7 parts, among them J1 GPIO_CONNECTOR, J2 BME680_CONNECTOR, J3 RFM95W_CONNECTOR

Commit message: modification of pcb
Connections:
- J1 pad 15: /GPIO22_GEN3 -> +3V3
- J1 pad 19: /GPIO10_SPI_MOSI -> +3V3
- J3 pad 4: /GPIO22_GEN3 -> +3V3
- J3 pad 7: /GPIO10_SPI_MOSI -> +3V3
Routing:
- net GND: track 80.6 -> 1.10 mm
- net /GPIO22_GEN3: track 36.0 -> 0.00 mm
- net +3V3: track 91.8 -> 125.5 mm
- net /GPIO10_SPI_MOSI: track 19.5 -> 0.00 mm
- net /GPIO25_GEN6: track 20.2 -> 18.1 mm
- net /GPIO11_SPI_SCLK: track 16.1 -> 17.4 mm
- net (no net): track 0.54 -> 0.00 mm
- added copper zone on B.Cu, net GND
- removed copper zone on B.Cu, net (none)

Commit message: modification of pcb
Parts:
- added R1: R, Resistor_SMD:R_1806_4516Metric, F.Cu at (154.1, 99.6)
- added R2: R, Resistor_SMD:R_1806_4516Metric, F.Cu at (154.1, 103.5)
- added R3: R, Resistor_SMD:R_1806_4516Metric, F.Cu at (160.4, 103.5)
- moved J2 15.3 mm to (131.2, 117.4), turned to 0 degrees
- moved J3 14.8 mm to (166.8, 118.7), turned to 0 degrees
- moved J1 0.21 mm to (126.1, 95.8)
Connections:
- J1 pad 15: +3V3 -> /GPIO22_GEN3
- J1 pad 19: +3V3 -> /GPIO10_SPI_MOSI
- J3 pad 4: +3V3 -> /GPIO22_GEN3
- J3 pad 6: /GPIO9_SPI_MISO -> Net-(J3-Pad6)
- J3 pad 7: +3V3 -> Net-(J3-Pad7)
Routing:
- net +3V3: track 125.5 -> 61.6 mm
- net GND: track 1.10 -> 44.3 mm
- net /GPIO22_GEN3: track 0.00 -> 37.4 mm
- net /GPIO9_SPI_MISO: track 17.4 -> 0.00 mm
- net Net-(J3-Pad7): track 0.00 -> 10.7 mm
- net /GPIO10_SPI_MOSI: track 0.00 -> 9.96 mm
- net Net-(J3-Pad6): track 0.00 -> 6.57 mm
- net /GPIO11_SPI_SCLK: track 17.4 -> 23.9 mm
- net /GPIO3_SCL1: track 11.3 -> 16.8 mm
- net Net-(R1-Pad1): track 0.00 -> 5.10 mm
- net /GPIO8_SPI_CE0_N: track 19.5 -> 16.9 mm
- net +5V: track 2.54 -> 0.00 mm
- net /GPIO25_GEN6: track 18.1 -> 19.4 mm
- added copper zone on F.Cu, net GND
- removed copper zone on B.Cu, net GND
